File: 74xx_pdp8_reg_mux_board/74xx_pdp8_reg_mux_board.sch (KiCad schematic (older format))
At the start: 54 parts, among them U18 74LS251, U19 74LS251, U20 74LS251, U21 74LS251, U22 74LS251, U23 74LS251, U24 74LS251, U25 74LS251, U26 74LS251, U27 74LS251, U28 74LS251, U29 74LS251

Commit message: Revised and tidied register mux schematic and 'pcb' layout.
Parts:
- removed C16, C17, C18, C19, C20, C21, C22, C23, C24, C25, C26, C27, C28, C29: 1uF, Capacitors_ThroughHole:C_Disc_D3_P2.5, symbol C_Small
- removed R1: R_Small, Discret:R1, symbol R_Small
- added P1, P2, P3, P4, P5, P6: DIL24, Socket_Strips:Socket_Strip_Straight_2x12, symbol DIL24
- U11, U3, U7: renamed from U?; footprint (none) -> Housings_DIP:DIP-14_W7.62mm
- renumbered U18 to U1, U25 to U10, U26 to U12, U27 to U13, U28 to U14, U29 to U15, U19 to U2, U20 to U4, U21 to U5, U22 to U6, U23 to U8, U24 to U9
Connections:
- net OUT0 is gone; now on net OUT_0: U1.5 (Z)
- net OUT1 is gone; now on net OUT_1: U2.5 (Z)
- net OUT2 is gone; now on net OUT_2: U4.5 (Z)
- net OUT3 is gone; now on net OUT_3: U5.5 (Z)
- net OUT4 is gone; now on net OUT_4: U6.5 (Z)
- net OUT8 is gone; now on net OUT_8: U12.5 (Z)
- net GND: now also U11.1 (E), U11.10 (E), U11.13 (E), U11.4 (E), U3.1 (E), U3.10 (E), U3.13 (E), U3.4 (E), U7.1 (E), U7.10 (E), U7.13 (E), U7.4 (E), P6.2 (P2)
- net S0: now also P6.16 (P16)
- net S1: now also P6.17 (P17)
- net S2: now also P6.18 (P18)
- net VCC: now also P6.1 (P1)
- net OUT_0: now reaches U3.2 (D)
- net OUT_0: now also P2.1 (P1)
- net OUT_BUF_0: now reaches U3.3 (O)
- net OUT_BUF_0: now also P4.1 (P1)
- net OUT_1: now reaches U3.5 (D)
- net OUT_1: now also P2.2 (P2)
- net OUT_BUF_1: now reaches U3.6 (O)
- net OUT_BUF_1: now also P4.2 (P2)
- net OUT_BUF_2: now reaches U3.8 (O)
- net OUT_BUF_2: now also P4.3 (P3)
- net OUT_2: now reaches U3.9 (D)
- net OUT_2: now also P2.3 (P3)
- net OUT_BUF_3: now reaches U3.11 (O)
- net OUT_BUF_3: now also P4.4 (P4)
- net OUT_3: now reaches U3.12 (D)
- net OUT_3: now also P2.4 (P4)
- net OUT_4: now reaches U7.2 (D)
- net OUT_4: now also P2.5 (P5)
- net OUT_BUF_4: now reaches U7.3 (O)
- net OUT_BUF_4: now also P4.5 (P5)
- net OUT_8: now reaches U11.2 (D)
- net OUT_8: now also P2.9 (P9)
- net OUT_BUF_8: now reaches U11.3 (O)
- net OUT_BUF_8: now also P4.9 (P9)
- net IN_F_4: now reaches U6.14 (I5)
- net IN_F_4: now also P5.17 (P17)
- net IN_F_5: now reaches U8.14 (I5)
- net IN_F_5: now also P5.18 (P18)
- net IN_F_6: now reaches U9.14 (I5)
- net IN_F_6: now also P5.19 (P19)
- net IN_F_7: now reaches U10.14 (I5)
- net IN_F_7: now also P5.20 (P20)
- net IN_F_8: now reaches U12.14 (I5)
- net IN_F_8: now also P5.21 (P21)
- net IN_F_9: now reaches U13.14 (I5)
- net IN_F_9: now also P5.22 (P22)
- net IN_F_10: now reaches U14.14 (I5)
- net IN_F_10: now also P5.23 (P23)
- net IN_F_11: now reaches U15.14 (I5)
- net IN_F_11: now also P5.24 (P24)
- net IN_F_0: now reaches U1.14 (I5)
- net IN_F_0: now also P5.13 (P13)
- net IN_F_1: now reaches U2.14 (I5)
- net IN_F_1: now also P5.14 (P14)
- net IN_F_2: now reaches U4.14 (I5)
- net IN_F_2: now also P5.15 (P15)
- net IN_F_3: now reaches U5.14 (I5)
- net IN_F_3: now also P5.16 (P16)
- net OUT10 renamed OUT_10
- net OUT_10: now also U11.9 (D), P2.11 (P11)
- net OUT11 renamed OUT_11
- net OUT_11: now also U11.12 (D), P2.12 (P12)
- net OUT5 renamed OUT_5
- net OUT_5: now also U7.5 (D), P2.6 (P6)
- net OUT6 renamed OUT_6
- net OUT_6: now also U7.9 (D), P2.7 (P7)
- net OUT7 renamed OUT_7
- net OUT_7: now also U7.12 (D), P2.8 (P8)
- net OUT9 renamed OUT_9
- net OUT_9: now also U11.5 (D), P2.10 (P10)
- net OUTa0 renamed IN_A_0
- net IN_A_0: now also P1.1 (P1)
- net OUTa1 renamed IN_A_1
- net IN_A_1: now also P1.2 (P2)
- net OUTa10 renamed IN_A_10
- net IN_A_10: now also P1.11 (P11)
- net OUTa11 renamed IN_A_11
- net IN_A_11: now also P1.12 (P12)
- net OUTa2 renamed IN_A_2
- net IN_A_2: now also P1.3 (P3)
- net OUTa3 renamed IN_A_3
- net IN_A_3: now also P1.4 (P4)
- net OUTa4 renamed IN_A_4
- net IN_A_4: now also P1.5 (P5)
- net OUTa5 renamed IN_A_5
- net IN_A_5: now also P1.6 (P6)
- net OUTa6 renamed IN_A_6
- net IN_A_6: now also P1.7 (P7)
- net OUTa7 renamed IN_A_7
- net IN_A_7: now also P1.8 (P8)
- net OUTa8 renamed IN_A_8
- net IN_A_8: now also P1.9 (P9)
- net OUTa9 renamed IN_A_9
- net IN_A_9: now also P1.10 (P10)
- net OUTb0 renamed IN_B_0
- net IN_B_0: now also P1.13 (P13)
- net OUTb1 renamed IN_B_1
- net IN_B_1: now also P1.14 (P14)
- net OUTb10 renamed IN_B_10
- net IN_B_10: now also P1.23 (P23)
- net OUTb11 renamed IN_B_11
- net IN_B_11: now also P1.24 (P24)
- net OUTb2 renamed IN_B_2
- net IN_B_2: now also P1.15 (P15)
- net OUTb3 renamed IN_B_3
- net IN_B_3: now also P1.16 (P16)
- net OUTb4 renamed IN_B_4
- net IN_B_4: now also P1.17 (P17)
- net OUTb5 renamed IN_B_5
- net IN_B_5: now also P1.18 (P18)
- net OUTb6 renamed IN_B_6
- net IN_B_6: now also P1.19 (P19)
- net OUTb7 renamed IN_B_7
- net IN_B_7: now also P1.20 (P20)
- net OUTb8 renamed IN_B_8
- net IN_B_8: now also P1.21 (P21)
- net OUTb9 renamed IN_B_9
- net IN_B_9: now also P1.22 (P22)
- net OUTc0 renamed IN_C_0
- net IN_C_0: now also P3.1 (P1); no longer U5.2 (I2)
- net OUTc1 renamed IN_C_1
- net IN_C_1: now also P3.2 (P2)
- net OUTc10 renamed IN_C_10
- net IN_C_10: now also P3.11 (P11)
- net OUTc11 renamed IN_C_11
- net IN_C_11: now also P3.12 (P12)
- net OUTc2 renamed IN_C_2
- net IN_C_2: now also P3.3 (P3)
- net OUTc4 renamed IN_C_4
- net IN_C_4: now also P3.5 (P5)
- net OUTc5 renamed IN_C_5
- net IN_C_5: now also P3.6 (P6)
- net OUTc6 renamed IN_C_6
- net IN_C_6: now also P3.7 (P7)
- net OUTc7 renamed IN_C_7
- net IN_C_7: now also P3.8 (P8)
- net OUTc8 renamed IN_C_8
- net IN_C_8: now also P3.9 (P9)
- net OUTc9 renamed IN_C_9
- net IN_C_9: now also P3.10 (P10)
- net OUTd0 renamed IN_D_0
- net IN_D_0: now also P3.13 (P13)
- net OUTd1 renamed IN_D_1
- net IN_D_1: now also P3.14 (P14)
- net OUTd10 renamed IN_D_10
- net IN_D_10: now also P3.23 (P23)
- net OUTd11 renamed IN_D_11
- net IN_D_11: now also P3.24 (P24)
- net OUTd2 renamed IN_D_2
- net IN_D_2: now also P3.15 (P15)
- net OUTd3 renamed IN_D_3
- net IN_D_3: now also P3.16 (P16)
- net OUTd4 renamed IN_D_4
- net IN_D_4: now also P3.17 (P17)
- net OUTd5 renamed IN_D_5
- net IN_D_5: now also P3.18 (P18)
- net OUTd6 renamed IN_D_6
- net IN_D_6: now also P3.19 (P19)
- net OUTd7 renamed IN_D_7
- net IN_D_7: now also P3.20 (P20)
- net OUTd8 renamed IN_D_8
- net IN_D_8: now also P3.21 (P21)
- net OUTd9 renamed IN_D_9
- net IN_D_9: now also P3.22 (P22)
- net OUTe0 renamed IN_E_0
- net IN_E_0: now also P5.1 (P1)
- net OUTe1 renamed IN_E_1
- net IN_E_1: now also P5.2 (P2)
- net OUTe10 renamed IN_E_10
- net IN_E_10: now also P5.11 (P11)
- net OUTe11 renamed IN_E_11
- net IN_E_11: now also P5.12 (P12)
- net OUTe2 renamed IN_E_2
- net IN_E_2: now also P5.3 (P3)
- net OUTe3 renamed IN_E_3
- net IN_E_3: now also P5.4 (P4)
- net OUTe4 renamed IN_E_4
- net IN_E_4: now also P5.5 (P5)
- net OUTe5 renamed IN_E_5
- net IN_E_5: now also P5.6 (P6)
- net OUTe6 renamed IN_E_6
- net IN_E_6: now also P5.7 (P7)
- net OUTe7 renamed IN_E_7
- net IN_E_7: now also P5.8 (P8)
- net OUTe8 renamed IN_E_8
- net IN_E_8: now also P5.9 (P9)
- net OUTe9 renamed IN_E_9
- net IN_E_9: now also P5.10 (P10)
- new net IN_C_3: P3.4 (P4), U5.2 (I2)
- new net OUT_BUF_10: P4.11 (P11), U11.8 (O)
- new net OUT_BUF_11: P4.12 (P12), U11.11 (O)
- new net OUT_BUF_5: P4.6 (P6), U7.6 (O)
- new net OUT_BUF_6: P4.7 (P7), U7.8 (O)
- new net OUT_BUF_7: P4.8 (P8), U7.11 (O)
- new net OUT_BUF_9: P4.10 (P10), U11.6 (O)
- no-connect marks 48 -> 36
Other:
- moved on the sheet: C1, C10, C11, C12, C13, C14, C15, C2, C3, C4, C5, C6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

Commit message: Lots of tidying up. Rationalised connectors at register board 'output' end. Connectors matched on register and mux boards.
Parts:
- removed P2, P4, P5: DIL24, Socket_Strips:Socket_Strip_Straight_2x12, symbol DIL24
- added P10, P11, P12, P13, P2, P4, P5, P9: DIL6, Socket_Strips:Socket_Strip_Straight_2x03, symbol DIL6
- added P7: DIL24, Socket_Strips:Socket_Strip_Straight_2x12, symbol DIL24
Connections:
- net OUT_0: now also P7.1 (P1)
- net OUT_1: now also P7.2 (P2)
- net OUT_10: now also P7.11 (P11)
- net OUT_11: now also P7.12 (P12)
- net OUT_2: now also P7.3 (P3)
- net OUT_3: now also P7.4 (P4)
- net OUT_4: now also P7.6 (P6)
- net OUT_5: now also P7.5 (P5)
- net OUT_6: now also P7.7 (P7)
- net OUT_7: now also P7.8 (P8)
- net OUT_8: now also P7.9 (P9)
- net OUT_9: now also P7.10 (P10)
- net OUT_BUF_0: now also P9.1 (P1)
- net OUT_BUF_1: now also P9.2 (P2)
- net OUT_BUF_10: now also P10.5 (P5)
- net OUT_BUF_11: now also P10.6 (P6)
- net OUT_BUF_2: now also P9.3 (P3)
- net OUT_BUF_3: now also P9.4 (P4)
- net OUT_BUF_4: now also P9.5 (P5)
- net OUT_BUF_5: now also P9.6 (P6)
- net OUT_BUF_6: now also P10.1 (P1)
- net OUT_BUF_7: now also P10.2 (P2)
- net OUT_BUF_8: now also P10.3 (P3)
- net OUT_BUF_9: now also P10.4 (P4)
- net IN_A_0 renamed IN_MA_0
- net IN_A_1 renamed IN_MA_1
- net IN_A_10 renamed IN_MA_10
- net IN_A_11 renamed IN_MA_11
- net IN_A_2 renamed IN_MA_2
- net IN_A_3 renamed IN_MA_3
- net IN_A_4 renamed IN_MA_4
- net IN_A_5 renamed IN_MA_5
- net IN_A_6 renamed IN_MA_6
- net IN_A_7 renamed IN_MA_7
- net IN_A_8 renamed IN_MA_8
- net IN_A_9 renamed IN_MA_9
- net IN_B_0 renamed IN_MD_0
- net IN_B_1 renamed IN_MD_1
- net IN_B_10 renamed IN_MD_10
- net IN_B_11 renamed IN_MD_11
- net IN_B_2 renamed IN_MD_2
- net IN_B_3 renamed IN_MD_3
- net IN_B_4 renamed IN_MD_4
- net IN_B_5 renamed IN_MD_5
- net IN_B_6 renamed IN_MD_6
- net IN_B_7 renamed IN_MD_7
- net IN_B_8 renamed IN_MD_8
- net IN_B_9 renamed IN_MD_9
- net IN_C_0 renamed IN_PC_0
- net IN_C_1 renamed IN_PC_1
- net IN_C_10 renamed IN_PC_10
- net IN_C_11 renamed IN_PC_11
- net IN_C_2 renamed IN_PC_2
- net IN_C_3 renamed IN_PC_3
- net IN_C_4 renamed IN_PC_4
- net IN_C_5 renamed IN_PC_5
- net IN_C_6 renamed IN_PC_6
- net IN_C_7 renamed IN_PC_7
- net IN_C_8 renamed IN_PC_8
- net IN_C_9 renamed IN_PC_9
- net IN_D_0 renamed IN_AC_0
- net IN_AC_0: now also P7.13 (P13); no longer U1.1 (I3)
- net IN_D_1 renamed IN_AC_1
- net IN_AC_1: now also P7.14 (P14); no longer U2.1 (I3)
- net IN_D_10 renamed IN_AC_10
- net IN_AC_10: now also P7.23 (P23); no longer U14.1 (I3)
- net IN_D_11 renamed IN_AC_11
- net IN_AC_11: now also P7.24 (P24); no longer U15.1 (I3)
- net IN_D_2 renamed IN_AC_2
- net IN_AC_2: now also P7.15 (P15); no longer U4.1 (I3)
- net IN_D_3 renamed IN_AC_3
- net IN_AC_3: now also P7.16 (P16); no longer U5.1 (I3)
- net IN_D_4 renamed IN_AC_4
- net IN_AC_4: now also P7.17 (P17); no longer U6.1 (I3)
- net IN_D_5 renamed IN_AC_5
- net IN_AC_5: now also P7.18 (P18); no longer U8.1 (I3)
- net IN_D_6 renamed IN_AC_6
- net IN_AC_6: now also P7.19 (P19); no longer U9.1 (I3)
- net IN_D_7 renamed IN_AC_7
- net IN_AC_7: now also P7.20 (P20); no longer U10.1 (I3)
- net IN_D_8 renamed IN_AC_8
- net IN_AC_8: now also P7.21 (P21); no longer U12.1 (I3)
- net IN_D_9 renamed IN_AC_9
- net IN_AC_9: now also P7.22 (P22); no longer U13.1 (I3)
- net IN_E_0 renamed IN_IOT1_0
- net IN_IOT1_0: now also P5.1 (P1)
- net IN_E_1 renamed IN_IOT1_1
- net IN_IOT1_1: now also P5.2 (P2)
- net IN_E_10 renamed IN_IOT1_10
- net IN_IOT1_10: now also P11.5 (P5)
- net IN_E_11 renamed IN_IOT1_11
- net IN_IOT1_11: now also P11.6 (P6)
- net IN_E_2 renamed IN_IOT1_2
- net IN_IOT1_2: now also P5.3 (P3)
- net IN_E_3 renamed IN_IOT1_3
- net IN_IOT1_3: now also P5.4 (P4)
- net IN_E_4 renamed IN_IOT1_4
- net IN_IOT1_4: now also P5.5 (P5)
- net IN_E_5 renamed IN_IOT1_5
- net IN_IOT1_5: now also P5.6 (P6)
- net IN_E_6 renamed IN_IOT1_6
- net IN_IOT1_6: now also P11.1 (P1)
- net IN_E_7 renamed IN_IOT1_7
- net IN_IOT1_7: now also P11.2 (P2)
- net IN_E_8 renamed IN_IOT1_8
- net IN_IOT1_8: now also P11.3 (P3)
- net IN_E_9 renamed IN_IOT1_9
- net IN_IOT1_9: now also P11.4 (P4)
- net IN_F_0 renamed IN_IOT2_0
- net IN_IOT2_0: now also P12.1 (P1)
- net IN_F_1 renamed IN_IOT2_1
- net IN_IOT2_1: now also P12.2 (P2)
- net IN_F_10 renamed IN_IOT2_10
- net IN_IOT2_10: now also P13.5 (P5)
- net IN_F_11 renamed IN_IOT2_11
- net IN_IOT2_11: now also P13.6 (P6)
- net IN_F_2 renamed IN_IOT2_2
- net IN_IOT2_2: now also P12.3 (P3)
- net IN_F_3 renamed IN_IOT2_3
- net IN_IOT2_3: now also P12.4 (P4)
- net IN_F_4 renamed IN_IOT2_4
- net IN_IOT2_4: now also P12.5 (P5)
- net IN_F_5 renamed IN_IOT2_5
- net IN_IOT2_5: now also P12.6 (P6)
- net IN_F_6 renamed IN_IOT2_6
- net IN_IOT2_6: now also P13.1 (P1)
- net IN_F_7 renamed IN_IOT2_7
- net IN_IOT2_7: now also P13.2 (P2)
- net IN_F_8 renamed IN_IOT2_8
- net IN_IOT2_8: now also P13.3 (P3)
- net IN_F_9 renamed IN_IOT2_9
- net IN_IOT2_9: now also P13.4 (P4)
- new net IN_SR_0: P2.1 (P1), U1.1 (I3)
- new net IN_SR_1: P2.2 (P2), U2.1 (I3)
- new net IN_SR_10: P4.5 (P5), U14.1 (I3)
- new net IN_SR_11: P4.6 (P6), U15.1 (I3)
- new net IN_SR_2: P2.3 (P3), U4.1 (I3)
- new net IN_SR_3: P2.6 (P6), U5.1 (I3)
- new net IN_SR_4: P2.5 (P5), U6.1 (I3)
- new net IN_SR_5: P2.4 (P4), U8.1 (I3)
- new net IN_SR_6: P4.1 (P1), U9.1 (I3)
- new net IN_SR_7: P4.2 (P2), U10.1 (I3)
- new net IN_SR_8: P4.3 (P3), U12.1 (I3)
- new net IN_SR_9: P4.4 (P4), U13.1 (I3)
Other:
- moved on the sheet: C1, C10, C11, C12, C13, C14, C15, C2, C3, C4, C5, C6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

Commit message: Big changes - elected to switch to board interconnections along one long edge only. Boards to connect to backplane via right-angled DIL connectors. Both register boards and register mux boards thusly modified.
Connections:
- net GND: now also U1.12 (I7), U1.13 (I6), U10.12 (I7), U10.13 (I6), U12.12 (I7), U12.13 (I6), U13.12 (I7), U13.13 (I6), U14.12 (I7), U14.13 (I6), U15.12 (I7), U15.13 (I6), U2.12 (I7), U2.13 (I6), U4.12 (I7), U4.13 (I6), U5.12 (I7), U5.13 (I6), U6.12 (I7), U6.13 (I6), U8.12 (I7), U8.13 (I6), U9.12 (I7), U9.13 (I6)
- no-connect marks 36 -> 12
Other:
- moved on the sheet: P10, P6, P9
